File: LVDS_Drvr/LVDS_Drvr.sch (KiCad schematic (older format))
At the start: 24 parts, among them M1 mosfet_n, M10 mosfet_n, M11 mosfet_p, M12 mosfet_n, M13 mosfet_n, M14 mosfet_n, M15 mosfet_p, M16 mosfet_n, M2 mosfet_n, M3 mosfet_n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

Commit message: new files update
Parts:
- added U5: IC, symbol IC
Connections:
- net Vocm: now also U5.1
- net Vdd: now reaches M11.3 (S), M11.4 (B), M15.3 (S), M15.4 (B), M5.3 (S), M5.4 (B), M6.3 (S), M6.4 (B), vdd1.1 (+)
- net Din: now reaches M1.2 (G), M4.2 (G), U1.~, v1.1 (+)
- net Din_bar: now reaches M2.2 (G), M3.2 (G), U2.~, v2.1 (+)
- net Vbias: now reaches M13.2 (G), M14.2 (G), vbias1.1 (+)
Changed lines of the file:
@@
 Connection ~ 6250 3400
 Wire Wire Line
-	6350 4250 6800 4250
+	6100 4250 6800 4250
 $Comp
 L DC vdd1
@@
 	6500 5300 6500 5500
 Wire Wire Line
-	900  1900 900  2200
+	900  1700 900  2200
 Wire Wire Line
 	900  3100 900  3300
@@
 $EndComp
 $Comp
+L GND #PWR3
+U 1 1 621B005D
+P 1550 5300
+F 0 "#PWR3" H 1550 5050 50  0001 C CNN
+F 1 "GND" H 1550 5150 50  0000 C CNN
+F 2 "" H 1550 5300 50  0001 C CNN
+F 3 "" H 1550 5300 50  0001 C CNN
+	1    1550 5300
+	1    0    0    -1
+$EndComp
+Wire Wire Line
+	900  5200 900  5300
+Wire Wire Line
+	1550 5200 1550 5300
+$Comp
+L plot_v1 U1
+U 1 1 621B0483
+P 1250 2800
+F 0 "U1" H 1250 3300 60  0000 C CNN
+F 1 "plot_v1" H 1450 3150 60  0000 C CNN
+F 2 "" H 1250 2800 60  0000 C CNN
+F 3 "" H 1250 2800 60  0000 C CNN
+	1    1250 2800
+	1    0    0    -1
+$EndComp
+$Comp
+L plot_v1 U2
+U 1 1 621B04E0
+P 1300 3650
+F 0 "U2" H 1300 4150 60  0000 C CNN
+F 1 "plot_v1" H 1500 4000 60  0000 C CNN
+F 2 "" H 1300 3650 60  0000 C CNN
+F 3 "" H 1300 3650 60  0000 C CNN
+	1    1300 3650
+	1    0    0    -1
+$EndComp
+Wire Wire Line
+	1250 2600 1250 3050
+Connection ~ 1250 3000
+Wire Wire Line
+	1300 3450 1300 3850
+Connection ~ 1300 3650
+$Comp
+L plot_v1 U3
+U 1 1 621B0790
+P 1950 3350
+F 0 "U3" H 1950 3850 60  0000 C CNN
+F 1 "plot_v1" H 2150 3700 60  0000 C CNN
+F 2 "" H 1950 3350 60  0000 C CNN
+F 3 "" H 1950 3350 60  0000 C CNN
+	1    1950 3350
+	1    0    0    -1
+$EndComp
+$Comp
+L plot_v1 U4
+U 1 1 621B07EF
+P 2500 3350
+F 0 "U4" H 2500 3850 60  0000 C CNN
+F 1 "plot_v1" H 2700 3700 60  0000 C CNN
+F 2 "" H 2500 3350 60  0000 C CNN
+F 3 "" H 2500 3350 60  0000 C CNN
+	1    2500 3350
+	1    0    0    -1
+$EndComp
+Wire Wire Line
+	1950 3150 1950 3500
+Connection ~ 1800 3300
+Wire Wire Line
+	2500 3150 2500 3500
+Connection ~ 2750 3300
+Wire Wire Line
+	1550 4300 1550 3850
+Wire Wire Line
+	1550 3850 1300 3850
+Wire Wire Line
+	900  4300 900  3850
+Wire Wire Line
+	900  3850 700  3850
+Wire Wire Line
+	700  3850 700  3550
+Wire Wire Line
+	700  3550 1150 3550
+Wire Wire Line
+	1150 3550 1150 3050
+Wire Wire Line
+	1150 3050 1250 3050
+Wire Wire Line
+	900  1900 7000 1900
+Wire Wire Line
+	5150 4250 4850 4250
+Wire Wire Line
+	4850 4250 4850 4000
+Wire Wire Line
+	4850 4000 6350 4000
+Wire Wire Line
+	6350 4000 6350 4250
+Wire Wire Line
+	4800 3400 3600 3400
+Wire Wire Line
+	3600 3400 3600 3300
+Wire Wire Line
+	7700 3400 8000 3400
+Wire Wire Line
+	8000 3400 8000 3100
+Wire Wire Line
+	8000 3100 3450 3100
+Wire Wire Line
+	3450 3100 3450 3350
+Wire Wire Line
+	3450 3350 1950 3350
+Connection ~ 1950 3300
+Wire Wire Line
+	1400 3000 1250 3000
+Wire Wire Line
+	3150 3650 3250 3650
+Wire Wire Line
+	3250 3650 3250 4050
+Wire Wire Line
+	3250 4050 800  4050
+Connection ~ 900  4050
+Wire Wire Line
+	1400 3650 1300 3650
+Wire Wire Line
+	3150 3000 3300 3000
+Wire Wire Line
+	3300 3000 3300 4000
+Wire Wire Line
+	3300 4000 1400 4000
+Connection ~ 1550 4000
+Text GLabel 1950 3500 3    60   Input ~ 0
+vob
+Text GLabel 2500 3500 3    60   Input ~ 0
+voa
+Connection ~ 1950 3350
+Connection ~ 2500 3300
+Text GLabel 700  4100 0    60   Input ~ 0
+Din
+Wire Wire Line
+	700  4100 800  4100
+Wire Wire Line
+	800  4100 800  4050
+Text GLabel 1400 4000 0    60   Input ~ 0
+Din_bar
+$Comp
 L GND #PWR2
 U 1 1 621B0021
@@
 $EndComp
 $Comp
-L GND #PWR3
-U 1 1 621B005D
-P 1550 5300
-F 0 "#PWR3" H 1550 5050 50  0001 C CNN
-F 1 "GND" H 1550 5150 50  0000 C CNN
-F 2 "" H 1550 5300 50  0001 C CNN
-F 3 "" H 1550 5300 50  0001 C CNN
-	1    1550 5300
-	1    0    0    -1
-$EndComp
-Wire Wire Line
-	900  5200 900  5300
-Wire Wire Line
-	1550 5200 1550 5300
-$Comp
-L plot_v1 U1
-U 1 1 621B0483
-P 1250 2800
-F 0 "U1" H 1250 3300 60  0000 C CNN
-F 1 "plot_v1" H 1450 3150 60  0000 C CNN
-F 2 "" H 1250 2800 60  0000 C CNN
-F 3 "" H 1250 2800 60  0000 C CNN
-	1    1250 2800
-	1    0    0    -1
-$EndComp
-$Comp
-L plot_v1 U2
-U 1 1 621B04E0
-P 1300 3650
-F 0 "U2" H 1300 4150 60  0000 C CNN
-F 1 "plot_v1" H 1500 4000 60  0000 C CNN
-F 2 "" H 1300 3650 60  0000 C CNN
-F 3 "" H 1300 3650 60  0000 C CNN
-	1    1300 3650
-	1    0    0    -1
-$EndComp
-Wire Wire Line
-	1250 2600 1250 3050
-Connection ~ 1250 3000
-Wire Wire Line
-	1300 3450 1300 3850
-Connection ~ 1300 3650
-$Comp
-L plot_v1 U3
-U 1 1 621B0790
-P 1950 3350
-F 0 "U3" H 1950 3850 60  0000 C CNN
-F 1 "plot_v1" H 2150 3700 60  0000 C CNN
-F 2 "" H 1950 3350 60  0000 C CNN
-F 3 "" H 1950 3350 60  0000 C CNN
-	1    1950 3350
-	1    0    0    -1
-$EndComp
-$Comp
-L plot_v1 U4
-U 1 1 621B07EF
-P 2500 3350
-F 0 "U4" H 2500 3850 60  0000 C CNN
-F 1 "plot_v1" H 2700 3700 60  0000 C CNN
-F 2 "" H 2500 3350 60  0000 C CNN
-F 3 "" H 2500 3350 60  0000 C CNN
-	1    2500 3350
-	1    0    0    -1
-$EndComp
-Wire Wire Line
-	1950 3150 1950 3500
-Connection ~ 1800 3300
-Wire Wire Line
-	2500 3150 2500 3500
-Connection ~ 2750 3300
-Wire Wire Line
-	1550 4300 1550 3850
-Wire Wire Line
-	1550 3850 1300 3850
-Wire Wire Line
-	900  4300 900  3850
-Wire Wire Line
-	900  3850 700  3850
-Wire Wire Line
-	700  3850 700  3550
-Wire Wire Line
-	700  3550 1150 3550
-Wire Wire Line
-	1150 3550 1150 3050
-Wire Wire Line
-	1150 3050 1250 3050
-Wire Wire Line
-	900  1900 7000 1900
-Wire Wire Line
-	5150 4250 4850 4250
-Wire Wire Line
-	4850 4250 4850 4000
-Wire Wire Line
-	4850 4000 6350 4000
-Wire Wire Line
-	6350 4000 6350 4250
-Wire Wire Line
-	4800 3400 3600 3400
-Wire Wire Line
-	3600 3400 3600 3300
-Wire Wire Line
-	7700 3400 8000 3400
-Wire Wire Line
-	8000 3400 8000 3100
-Wire Wire Line
-	8000 3100 3450 3100
-Wire Wire Line
-	3450 3100 3450 3350
-Wire Wire Line
-	3450 3350 1950 3350
-Connection ~ 1950 3300
-Wire Wire Line
-	1400 3000 1250 3000
-Wire Wire Line
-	3150 3650 3250 3650
-Wire Wire Line
-	3250 3650 3250 4050
-Wire Wire Line
-	3250 4050 900  4050
-Connection ~ 900  4050
-Wire Wire Line
-	1400 3650 1300 3650
-Wire Wire Line
-	3150 3000 3300 3000
-Wire Wire Line
-	3300 3000 3300 4000
-Wire Wire Line
-	3300 4000 1550 4000
-Connection ~ 1550 4000
-Text GLabel 1950 3500 3    60   Input ~ 0
-vob
-Text GLabel 2500 3500 3    60   Input ~ 0
-voa
-Connection ~ 1950 3350
-Connection ~ 2500 3300
+L IC U5
+U 1 1 6234A653
+P 6250 3100
+F 0 "U5" H 6550 3250 60  0000 C CNN
+F 1 "IC" H 6500 3450 60  0000 C CNN
+F 2 "" H 6250 3100 60  0000 C CNN
+F 3 "" H 6250 3100 60  0000 C CNN
+	1    6250 3100
+	1    0    0    -1
+$EndComp
+Wire Wire Line
+	6450 3050 6250 3050
+Connection ~ 6250 3050
+Text GLabel 6100 4250 0    60   Input ~ 0
+Vbias
+Connection ~ 6350 4250
+Text GLabel 900  1700 1    60   Input ~ 0
+Vdd
+Connection ~ 900  1900
 $EndSCHEMATC
